File: timer_remote.sch (EAGLE design)
At the start: 27 parts, among them J1 120VAC, J2 Low Volt Relay, K1 G5LE-14-DC5, K2 G5LE-14-DC5, Q1 DMN2053UVT

Commit message: Sent to fab.
Other:
- note added: "D3/R8 and D4/R9 are optional on-board indicators for the relays."
- moved on the sheet: A1, A2, C1, C2, D1, D2, D3, D4, J1, J2, JP1, JP2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

Commit message: Minor tweaks to PCB traces, update README, BoM, images.
Other:
- note added: "K2 is optional and intended for low-voltage use only."
Changed lines of the file:
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@@
 <text x="78.74" y="55.88" size="2.54" layer="94">D3/R8 and D4/R9 are optional
 on-board indicators for the relays.</text>
+<text x="187.96" y="55.88" size="2.54" layer="94">K2 is optional and intended
+for low-voltage use only.</text>
 </plain>
 <instances>
